File: Pro Micro FSR PCB.kicad_pcb (KiCad board)
At the start: 2 copper layers, 48 x 48 mm, 25 parts, among them J1 Conn_01x02_Pin, J2 Conn_01x02_Pin, J3 Conn_01x02_Pin, J4 Conn_01x02_Pin, J5 Conn_01x02_Pin, J6 Conn_01x02_Pin, J7 Conn_01x02_Pin, J8 Conn_01x02_Pin, U1 ProMicro

Commit message: Add files via upload
Parts:
- removed R1, R2, R3, R4, R5, R6, R7, R8: 1kOhm, Resistor_THT:R_Axial_DIN0204_L3.6mm_D1.6mm_P1.90mm_Vertical
- renumbered J8 to A0, J7 to A1, J6 to A2, J5 to A3, J4 to A6, J3 to A7, J2 to A8, J1 to A9
Connections:
- A0 pad 2: A9 -> A0
- A1 pad 2: A8 -> A1
- A2 pad 2: A7 -> A2
- A3 pad 2: A6 -> A3
- A6 pad 2: A3 -> A6
- A7 pad 2: A2 -> A7
- A8 pad 2: A1 -> A8
- A9 pad 2: A0 -> A9
